File: Debugger_port.kicad_sch (KiCad schematic)
At the start: 5 parts, among them J10 Conn_01x06_Female

Commit message: pcb is in progress, finishing H-bridge layout
Parts:
- D75, D76, D77, D78: footprint Diode_SMD:D_SMB -> _Diodes:SM2T3V3A
Changed lines of the file:
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@@
       (effects (font (size 1.27 1.27)) (justify left) hide)
     )
-    (property "Footprint" "Diode_SMD:D_SMB" (id 2) (at 146.05 110.49 0)
+    (property "Footprint" "_Diodes:SM2T3V3A" (id 2) (at 146.05 110.49 0)
       (effects (font (size 1.27 1.27)) hide)
     )
@@
       (effects (font (size 1.27 1.27)) (justify left) hide)
     )
-    (property "Footprint" "Diode_SMD:D_SMB" (id 2) (at 149.86 110.49 0)
+    (property "Footprint" "_Diodes:SM2T3V3A" (id 2) (at 149.86 110.49 0)
       (effects (font (size 1.27 1.27)) hide)
     )
@@
       (effects (font (size 1.27 1.27)) (justify left) hide)
     )
-    (property "Footprint" "Diode_SMD:D_SMB" (id 2) (at 153.67 110.49 0)
+    (property "Footprint" "_Diodes:SM2T3V3A" (id 2) (at 153.67 110.49 0)
       (effects (font (size 1.27 1.27)) hide)
     )
@@
       (effects (font (size 1.27 1.27)) (justify left))
     )
-    (property "Footprint" "Diode_SMD:D_SMB" (id 2) (at 142.24 110.49 0)
+    (property "Footprint" "_Diodes:SM2T3V3A" (id 2) (at 142.24 110.49 0)
       (effects (font (size 1.27 1.27)) hide)
     )

Commit message: added power loss detection, preparing for new pcb layout
Parts:
- D75, D76, D77, D78: footprint _Diodes:SM2T3V3A -> Diode_SMD:D_SMB
Changed lines of the file:
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@@
       (effects (font (size 1.27 1.27)) (justify left) hide)
     )
-    (property "Footprint" "_Diodes:SM2T3V3A" (id 2) (at 146.05 110.49 0)
+    (property "Footprint" "Diode_SMD:D_SMB" (id 2) (at 146.05 110.49 0)
       (effects (font (size 1.27 1.27)) hide)
     )
@@
       (effects (font (size 1.27 1.27)) (justify left) hide)
     )
-    (property "Footprint" "_Diodes:SM2T3V3A" (id 2) (at 149.86 110.49 0)
+    (property "Footprint" "Diode_SMD:D_SMB" (id 2) (at 149.86 110.49 0)
       (effects (font (size 1.27 1.27)) hide)
     )
@@
       (effects (font (size 1.27 1.27)) (justify left) hide)
     )
-    (property "Footprint" "_Diodes:SM2T3V3A" (id 2) (at 153.67 110.49 0)
+    (property "Footprint" "Diode_SMD:D_SMB" (id 2) (at 153.67 110.49 0)
       (effects (font (size 1.27 1.27)) hide)
     )
@@
       (effects (font (size 1.27 1.27)) (justify left))
     )
-    (property "Footprint" "_Diodes:SM2T3V3A" (id 2) (at 142.24 110.49 0)
+    (property "Footprint" "Diode_SMD:D_SMB" (id 2) (at 142.24 110.49 0)
       (effects (font (size 1.27 1.27)) hide)
     )
