File: SPI_port.kicad_sch (KiCad schematic)
At the start: 4 parts, among them J12 Conn_01x06_Female, J27 RJ12_Shielded

Commit message: remove all DRC place 3v3 caps added 3v3 vias added more new descriptions
Parts:
- removed D100, D98: AOZ8211, _Diodes:AOZ8211, symbol _Diodes:AOZ8211
- added D100, D98: UCLAMP3301D.TCT, _Diodes:UCLAMP3301D.TCT, symbol _Diodes:UCLAMP3301D.TCT
Connections:
- net +3V3: now also D100.1, D98.1
- net GND: now also D100.2, D98.2
Changed lines of the file:
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@@
     (pin "6")
+  )
+  (symbol (lib_id "_Diodes:UCLAMP3301D.TCT") (at 144.78 107.95 0) (unit 1)
+    (in_bom yes) (on_board yes)
+    (property "Reference" "D98" (id 0) (at 148.59 98.7355 0)
+      (effects (font (size 1.27 1.27)) (justify left))
+    )
+    (property "Value" "UCLAMP3301D.TCT" (id 1) (at 137.16 113.03 90)
+      (effects (font (size 1.27 1.27)) (justify left))
+    )
+    (property "Footprint" "_Diodes:UCLAMP3301D.TCT" (id 2) (at 144.78 107.95 0)
+      (effects (font (size 1.27 1.27)) hide)
+    )
+    (property "Datasheet" "" (id 3) (at 144.78 107.95 0)
+      (effects (font (size 1.27 1.27)) hide)
+    )
+    (pin "1")
+    (pin "2")
   )
   (symbol (lib_id "power:GND") (at 207.01 88.9 90) (unit 1)
@@
     )
     (pin "1")
+  )
+  (symbol (lib_id "_Diodes:UCLAMP3301D.TCT") (at 209.55 106.68 0) (unit 1)
+    (in_bom yes) (on_board yes)
+    (property "Reference" "D100" (id 0) (at 213.36 97.4655 0)
+      (effects (font (size 1.27 1.27)) (justify left))
+    )
+    (property "Value" "UCLAMP3301D.TCT" (id 1) (at 214.63 116.84 90)
+      (effects (font (size 1.27 1.27)) (justify left))
+    )
+    (property "Footprint" "_Diodes:UCLAMP3301D.TCT" (id 2) (at 209.55 106.68 0)
+      (effects (font (size 1.27 1.27)) hide)
+    )
+    (property "Datasheet" "" (id 3) (at 209.55 106.68 0)
+      (effects (font (size 1.27 1.27)) hide)
+    )
+    (pin "1")
+    (pin "2")
   )
   (symbol (lib_id "power:GND") (at 194.31 105.41 0) (unit 1)
@@
     (pin "1")
   )
-  (symbol (lib_id "_Diodes:AOZ8211") (at 142.24 100.33 90) (unit 1)
-    (in_bom yes) (on_board yes) (fields_autoplaced)
-    (property "Reference" "D98" (id 0) (at 147.32 99.0599 90)
-      (effects (font (size 1.27 1.27)) (justify right))
-    )
-    (property "Value" "AOZ8211" (id 1) (at 147.32 101.5999 90)
-      (effects (font (size 1.27 1.27)) (justify right))
-    )
-    (property "Footprint" "_Diodes:AOZ8211" (id 2) (at 142.24 100.33 0)
-      (effects (font (size 1.27 1.27)) hide)
-    )
-    (property "Datasheet" "" (id 3) (at 142.24 100.33 0)
-      (effects (font (size 1.27 1.27)) hide)
-    )
-    (pin "1")
-    (pin "2")
-  )
   (symbol (lib_id "power:GND") (at 209.55 105.41 0) (unit 1)
     (in_bom yes) (on_board yes) (fields_autoplaced)
@@
     (pin "1")
   )
-  (symbol (lib_id "_Diodes:AOZ8211") (at 207.01 99.06 90) (unit 1)
-    (in_bom yes) (on_board yes) (fields_autoplaced)
-    (property "Reference" "D100" (id 0) (at 212.09 97.7899 90)
-      (effects (font (size 1.27 1.27)) (justify right))
-    )
-    (property "Value" "AOZ8211" (id 1) (at 212.09 100.3299 90)
-      (effects (font (size 1.27 1.27)) (justify right))
-    )
-    (property "Footprint" "_Diodes:AOZ8211" (id 2) (at 207.01 99.06 0)
-      (effects (font (size 1.27 1.27)) hide)
-    )
-    (property "Datasheet" "" (id 3) (at 207.01 99.06 0)
-      (effects (font (size 1.27 1.27)) hide)
-    )
-    (pin "1")
-    (pin "2")
-  )
   (symbol (lib_id "_Connectors:RJ12_Shielded") (at 194.31 86.36 0) (unit 1)
