File: Power_supplies.kicad_sch (KiCad schematic)
At the start: 59 parts, among them J2 DG35C-B-02P, T1 AOSP21357, T2 MJD32C, U3 MC34063, U31 AP331A, U4 MC34063, U5 TLV70233_SOT23-5

Commit message: pcb commit repaired after diodes footprints errors
Parts:
- U31: footprint (none) -> _IntegratedCircuits:AP331A
Changed lines of the file:
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@@
       (effects (font (size 1.27 1.27)) (justify left))
     )
-    (property "Footprint" "" (id 2) (at 21.59 157.48 0)
+    (property "Footprint" "_IntegratedCircuits:AP331A" (id 2) (at 21.59 157.48 0)
       (effects (font (size 1.27 1.27)) hide)
     )
@@
     (property "Reference" "U31" (id 0) (at 64.77 147.32 0))
     (property "Value" "AP331A" (id 1) (at 64.77 149.86 0))
-    (property "Footprint" "" (id 2) (at 64.77 157.48 0)
-      (effects (font (size 1.27 1.27)) hide)
-    )
+    (property "Footprint" "_IntegratedCircuits:AP331A" (id 2) (at 64.77 157.48 0)
+      (effects (font (size 1.27 1.27)) hide)
+    )
