File: H_bridge.kicad_sch (KiCad schematic)
At the start: 48 parts, among them J1 Conn_01x02_Female, J9 Conn_01x03_Female, SW1 SW_SPST, T3 AOD4132, T4 AOD4132, T5 AOD4132, T6 AOD4132, U1 IR2104, U2 IR2104, U35 AP331A

Commit message: remove all DRC place 3v3 caps added 3v3 vias added more new descriptions
Parts:
- gave numbers to parts that had none: 1
Changed lines of the file:
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@@
   (symbol (lib_id "Connector:TestPoint") (at 130.81 162.56 180) (unit 1)
     (in_bom yes) (on_board yes)
-    (property "Reference" "TP?" (id 0) (at 129.54 167.64 0)
+    (property "Reference" "TP24" (id 0) (at 129.54 167.64 0)
       (effects (font (size 1.27 1.27)) (justify right))
     )
